File: PCB/_autosave-ESP_Windowsensor.sch (KiCad schematic (older format))
At the start: 22 parts, among them IC1 ATtiny13A-SSU, IC2 ESP-07, J1 AVR-ISP-6, J2 Conn_01x04_Female, Q1 IRLML6244, Q2 IRF3708, SW1 SW_Reed_SPDT, SW2 SW_Push, SW3 SW_Push

Commit message: Add files via upload
upload board rev 0.1
Parts:
- renumbered WIFI_RESET to WIFI_RESET1
Changed lines of the file:
@@
 	2950 5550 2950 6150
 $Comp
-L Jumper:SolderJumper_2_Open WIFI_RESET
+L Jumper:SolderJumper_2_Open WIFI_RESET1
 U 1 1 605B2A13
 P 10200 2250
-F 0 "WIFI_RESET" H 10154 2318 50  0000 L CNN
+F 0 "WIFI_RESET1" H 10154 2318 50  0000 L CNN
 F 1 "SolderJumper_2_Open" V 10245 2318 50  0001 L CNN
 F 2 "Jumper:SolderJumper-2_P1.3mm_Open_RoundedPad1.0x1.5mm" H 10200 2250 50  0001 C CNN
